File: eagle/oak_pcb.brd (EAGLE design)
At the start: 90.8 x 29.5 mm, 15 parts

Commit message: Board update, fixed some unfortunate mistakes on my part.
The oak only has a single Analog pin, I attached the sensor to one of
the digital pins. I can bodge the existing boards, but I’ve chosen to
order new boards anyway. So this will be version 2.0, also containing a
Ground pin for the UART connection as well as bigger holes for the IR
sensor and a jumper to set the module in ‘bootloader’ mode.
Parts:
- added JP5: (no value), SparkFun-Connectors:1X03_LOCK
- JP4: device SparkFun-Connectors:1X02_LOCK -> SparkFun-Connectors:1X03_LOCK
- R1, R2: device SparkFun-Passives:AXIAL-0.5 -> SparkFun-Passives:AXIAL-0.4
- moved JP4 12.7 mm to (59.7, 12.7)
- moved R1 11.4 mm to (45.7, 22.9), turned to 0 degrees
- moved R2 6.48 mm to (45.7, 12.7), turned to 0 degrees
- turned OS1 to 0 degrees
Connections:
- removed net SCL: JP2.4, JP3.3
- new net SCL_OLED: JP3.3, JP4.1
- new net SCL_PIN: JP2.4, JP4.2
- net GND: now also JP4.3, JP5.3
- net RX: now also JP5.2; no longer JP4.2
- net SENSE: now also JP1.3; no longer JP2.7
- net TX: now also JP5.1; no longer JP4.1
Routing:
- net SCL: track 29.4 -> 0.00 mm
- net SCL_OLED: track 0.00 -> 25.8 mm
- net SCL_PIN: track 0.00 -> 3.88 mm
- net N$3: track 11.7 -> 8.15 mm
- net VCC_3V3: track 141.6 -> 139.1 mm, vias 2 -> 3
- net RX: track 16.2 -> 14.6 mm
- net TX: track 14.2 -> 15.3 mm
Other:
- board text added: "1 2 3"
- board text added: "JP4: 1-2 BOOTLD 2-3 NORMAL JP5: GND, Rx, Tx"
- board text added: "V2.0"
- board text added: "https://github.com /DJFliX/OakPowerBoard"
