File: eagle/oak_pcb.sch (EAGLE design)
At the start: 15 parts

Commit message: Board update, fixed some unfortunate mistakes on my part.
The oak only has a single Analog pin, I attached the sensor to one of
the digital pins. I can bodge the existing boards, but I’ve chosen to
order new boards anyway. So this will be version 2.0, also containing a
Ground pin for the UART connection as well as bigger holes for the IR
sensor and a jumper to set the module in ‘bootloader’ mode.
Parts:
- added JP5: (no value), SparkFun-Connectors:M03LOCK
- JP4: device SparkFun-Connectors:M02LOCK -> SparkFun-Connectors:M03LOCK
- R1, R2: device SparkFun-Passives:RESISTORPTH-1/2W -> SparkFun-Passives:RESISTORPTH-1/4W
Connections:
- removed net SCL: JP2.4, JP3.3
- new net SCL_OLED: JP3.3, JP4.1
- new net SCL_PIN: JP2.4, JP4.2
- net GND: now also JP4.3, JP5.3
- net RX: now also JP5.2; no longer JP4.2
- net SENSE: now also JP1.3; no longer JP2.7
- net TX: now also JP5.1; no longer JP4.1
Changed lines of the file:
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@@
 <part name="JP2" library="SparkFun-Connectors" deviceset="M09" device="LOCK"/>
 <part name="OS1" library="tcrt5000" deviceset="TCRT5000" device=""/>
-<part name="R1" library="SparkFun-Passives" deviceset="RESISTOR" device="PTH-1/2W" value="10K"/>
+<part name="R1" library="SparkFun-Passives" deviceset="RESISTOR" device="PTH-1/4W" value="10K"/>
 <part name="GND1" library="SparkFun-Aesthetics" deviceset="GND" device=""/>
-<part name="R2" library="SparkFun-Passives" deviceset="RESISTOR" device="PTH-1/2W" value="330"/>
+<part name="R2" library="SparkFun-Passives" deviceset="RESISTOR" device="PTH-1/4W" value="330"/>
 <part name="GND2" library="SparkFun-Aesthetics" deviceset="GND" device=""/>
 <part name="JP3" library="SparkFun-Connectors" deviceset="M04" device="LOCK"/>
-<part name="JP4" library="SparkFun-Connectors" deviceset="M02" device="LOCK"/>
 <part name="S1" library="SparkFun-Electromechanical" deviceset="SWITCH-MOMENTARY-2" device="PTH"/>
 <part name="S2" library="SparkFun-Electromechanical" deviceset="SWITCH-MOMENTARY-2" device="PTH"/>
@@
 <part name="R6" library="SparkFun-Passives" deviceset="RESISTOR" device="PTH-1/4W" value="10K"/>
 <part name="GND3" library="SparkFun-Aesthetics" deviceset="GND" device=""/>
+<part name="JP5" library="SparkFun-Connectors" deviceset="M03" device="LOCK"/>
+<part name="JP4" library="SparkFun-Connectors" deviceset="M03" device="LOCK"/>
 </parts>
 <sheets>
@@
 <instance part="GND2" gate="1" x="25.4" y="60.96"/>
 <instance part="JP3" gate="G$1" x="30.48" y="104.14"/>
-<instance part="JP4" gate="G$1" x="93.98" y="109.22" rot="R270"/>
 <instance part="S1" gate="G$1" x="149.86" y="124.46"/>
 <instance part="S2" gate="G$1" x="149.86" y="116.84"/>
@@
 <instance part="R6" gate="G$1" x="132.08" y="101.6"/>
 <instance part="GND3" gate="1" x="114.3" y="88.9"/>
+<instance part="JP5" gate="G$1" x="81.28" y="109.22" rot="R270"/>
+<instance part="JP4" gate="G$1" x="27.94" y="88.9"/>
 </instances>
 <busses>
@@
 <junction x="114.3" y="101.6"/>
 <pinref part="GND3" gate="1" pin="GND"/>
+</segment>
+<segment>
+<pinref part="JP5" gate="G$1" pin="3"/>
+<wire x1="83.82" y1="101.6" x2="83.82" y2="96.52" width="0.1524" layer="91"/>
+<label x="83.82" y="96.52" size="1.778" layer="95" rot="R90"/>
+</segment>
+<segment>
+<pinref part="JP4" gate="G$1" pin="3"/>
+<wire x1="35.56" y1="91.44" x2="48.26" y2="91.44" width="0.1524" layer="91"/>
+<label x="43.18" y="91.44" size="1.778" layer="95"/>
 </segment>
 </net>
@@
 </segment>
 <segment>
-<pinref part="JP2" gate="G$1" pin="7"/>
-<wire x1="68.58" y1="43.18" x2="83.82" y2="43.18" width="0.1524" layer="91"/>
-<label x="78.74" y="43.18" size="1.778" layer="95"/>
+<pinref part="JP1" gate="G$1" pin="3"/>
+<wire x1="43.18" y1="43.18" x2="30.48" y2="43.18" width="0.1524" layer="91"/>
+<label x="30.48" y="43.18" size="1.778" layer="95"/>
 </segment>
 </net>
@@
 </segment>
 </net>
-<net name="SCL" class="0">
-<segment>
-<pinref part="JP3" gate="G$1" pin="3"/>
-<wire x1="35.56" y1="106.68" x2="48.26" y2="106.68" width="0.1524" layer="91"/>
-<label x="43.18" y="106.68" size="1.778" layer="95"/>
-</segment>
-<segment>
-<pinref part="JP2" gate="G$1" pin="4"/>
-<wire x1="68.58" y1="35.56" x2="83.82" y2="35.56" width="0.1524" layer="91"/>
-<label x="78.74" y="35.56" size="1.778" layer="95"/>
-</segment>
-</net>
 <net name="SDA" class="0">
 <segment>
@@
 </segment>
 <segment>
-<pinref part="JP4" gate="G$1" pin="1"/>
-<wire x1="93.98" y1="101.6" x2="93.98" y2="96.52" width="0.1524" layer="91"/>
-<label x="93.98" y="99.06" size="1.778" layer="95" rot="R90"/>
+<pinref part="JP5" gate="G$1" pin="1"/>
+<wire x1="78.74" y1="101.6" x2="78.74" y2="96.52" width="0.1524" layer="91"/>
+<label x="78.74" y="96.52" size="1.778" layer="95" rot="R90"/>
 </segment>
 </net>
@@
 </segment>
 <segment>
-<pinref part="JP4" gate="G$1" pin="2"/>
-<wire x1="96.52" y1="101.6" x2="96.52" y2="96.52" width="0.1524" layer="91"/>
-<label x="96.52" y="99.06" size="1.778" layer="95" rot="R90"/>
+<pinref part="JP5" gate="G$1" pin="2"/>
+<wire x1="81.28" y1="101.6" x2="81.28" y2="96.52" width="0.1524" layer="91"/>
+<label x="81.28" y="96.52" size="1.778" layer="95" rot="R90"/>
 </segment>
 </net>
@@
 </segment>
 </net>
+<net name="SCL_PIN" class="0">
+<segment>
+<pinref part="JP4" gate="G$1" pin="2"/>
+<wire x1="35.56" y1="88.9" x2="48.26" y2="88.9" width="0.1524" layer="91"/>
+<label x="43.18" y="88.9" size="1.778" layer="95"/>
+</segment>
+<segment>
+<pinref part="JP2" gate="G$1" pin="4"/>
+<wire x1="68.58" y1="35.56" x2="83.82" y2="35.56" width="0.1524" layer="91"/>
+<label x="78.74" y="35.56" size="1.778" layer="95"/>
+</segment>
+</net>
+<net name="SCL_OLED" class="0">
+<segment>
+<pinref part="JP4" gate="G$1" pin="1"/>
+<wire x1="35.56" y1="86.36" x2="48.26" y2="86.36" width="0.1524" layer="91"/>
+<label x="43.18" y="86.36" size="1.778" layer="95"/>
+</segment>
+<segment>
+<pinref part="JP3" gate="G$1" pin="3"/>
+<wire x1="35.56" y1="106.68" x2="48.26" y2="106.68" width="0.1524" layer="91"/>
+<label x="43.18" y="106.68" size="1.778" layer="95"/>
+</segment>
+</net>
